Commit message: Modifty tinker description for ros2 control

File: src/tinker_description/src/description/tinker.urdf.xacro (robot description, xacro)
@@ -28,5 +28,5 @@
   <link name="base_link_inertial">
     <inertial>
-      <origin xyz="0 0 0.3" rpy="0 0 0" />
+      <origin xyz="0 0 0.4" rpy="0 0 0" />
       <mass value="15" />
       <inertia ixx="0.3" ixy="0" ixz="0" iyy="0.3" iyz="0" izz="0.3" />
@@ -36,5 +36,5 @@
     <parent link="base_link" />
     <child link="base_link_inertial" />
-    <origin xyz="0 0 0" />
+    <origin xyz="0.02 0 0" />
   </joint>
   <link name="laser" />
@@ -45,3 +45,18 @@
     <origin xyz="${urg_front_trans_xyz}" />
   </joint>
+  <!-- Model used for real control, no wheel inertia needed -->
+  <xacro:macro name="wheel_gen" params="name prefix_1 prefix_2">
+    <joint name="${name}_wheel_joint" type="continuous">
+      <origin rpy="0 0 ${(prefix_2 + 1) / 2 *pi}" xyz="${prefix_1*0.22} ${prefix_2*0.17} 0.07"/>
+      <parent link="base_link_inertial"/>
+      <child link="${name}_wheel_link"/>
+      <limit effort="1.5" velocity="20"/>
+      <axis xyz="0 ${-1 * prefix_2} 0"/>
+    </joint>
+    <link name="${name}_wheel_link"/>
+  </xacro:macro>
+  <xacro:wheel_gen name="fl" prefix_1="1" prefix_2="1" />
+  <xacro:wheel_gen name="fr" prefix_1="1" prefix_2="-1" />
+  <xacro:wheel_gen name="rl" prefix_1="-1" prefix_2="1" />
+  <xacro:wheel_gen name="rr" prefix_1="-1" prefix_2="-1" />
 </robot>
